File: RPi-OLED-Adapter.kicad_pcb (KiCad board)
At the start: 4 copper layers, 65 x 56 mm, 35 parts, among them J1 GPIO, J2 DSI IN, J9 OLED_H497TLB01, U1 CAT24C256, U2 TCA9800, U3 TPS76318, U4 TPS22917DBV

Commit message: Create files for v1.1.0 release
Other:
- board text added: "${TITLE} ${COMPANY} ${REVISION}"
