File: RPi-OLED-Adapter.kicad_sch (KiCad schematic)
At the start: 31 parts, among them J1 GPIO, J2 DSI IN, J9 OLED_H497TLB01, U1 CAT24C256, U2 TCA9800, U3 TPS76318, U4 TPS22917DBV

Commit message: Create files for v1.1.0 release
Parts:
- J1: LCSC Part # (none) -> C25503128; MPN (none) -> 2541FV-2x20P-B
- J9: value OLED_H497TLB01 -> H499TLB01
Other:
- note removed: "Additional pin functions: https://pinout.xyz/"
- company: (none) -> ${COMPANY}
- title: (none) -> ${TITLE}
